Commit message: Added sensors

File: src/my_robot/urdf/my_robot.xacro (robot description, xacro)
@@ -1,57 +1,162 @@
-<?xml version='1.0'?>
+<?xml version="1.0"?>
 <robot name="my_robot" xmlns:xacro="http://www.ros.org/wiki/xacro">
-  <link name="robot_footprint"></link>
-  <joint name="robot_footprint_joint" type="fixed">
-    <origin xyz="0 0 0" rpy="0 0 0" />
-    <parent link="robot_footprint"/>
-    <child link="chassis" />
-  </joint>
-  <link name='chassis'>
-    <pose>0 0 0.1 0 0 0</pose>
-    <inertial>
-      <mass value="15.0"/>
-      <origin xyz="0.0 0 0" rpy=" 0 0 0"/>
-      <inertia
-          ixx="0.1" ixy="0" ixz="0"
-          iyy="0.1" iyz="0"
-          izz="0.1"
-      />
-    </inertial>
-    <collision name='collision'>
-      <origin xyz="0 0 0" rpy=" 0 0 0"/>
-      <geometry>
-        <box size=".4 .2 .1"/>
-      </geometry>
-    </collision>
-    <visual name='chassis_visual'>
-      <origin xyz="0 0 0" rpy=" 0 0 0"/>
-      <geometry>
-        <box size=".4 .2 .1"/>
-      </geometry>
-    </visual>
-    <collision name='back_caster_collision'>
-      <origin xyz="-0.15 0 -0.05" rpy=" 0 0 0"/>
-      <geometry>
-        <sphere radius="0.0499"/>
-      </geometry>
-    </collision>
-    <visual name='back_caster_visual'>
-      <origin xyz="-0.15 0 -0.05" rpy=" 0 0 0"/>
-      <geometry>
-        <sphere radius="0.05"/>
-      </geometry>
-    </visual>
-    <collision name='front_caster_collision'>
-      <origin xyz="0.15 0 -0.05" rpy=" 0 0 0"/>
-      <geometry>
-        <sphere radius="0.0499"/>
-      </geometry>
-    </collision>
-    <visual name='front_caster_visual'>
-      <origin xyz="0.15 0 -0.05" rpy=" 0 0 0"/>
-      <geometry>
-        <sphere radius="0.05"/>
-      </geometry>
-    </visual>
-  </link>
+	<include filename="$(find my_robot)/urdf/my_robot.gazebo" />
+	<link name="robot_footprint">
+	</link>
+	<joint name="robot_footprint_joint" type="fixed">
+		<origin xyz="0 0 0" rpy="0 0 0" />
+		<parent link="robot_footprint" />
+		<child link="chassis" />
+	</joint>
+	<link name="chassis">
+		<pose>
+			0 0 0.1 0 0 0
+		</pose>
+		<inertial>
+			<mass value="15.0" />
+			<origin xyz="0.0 0 0" rpy=" 0 0 0" />
+			<inertia ixx="0.1" ixy="0" ixz="0" iyy="0.1" iyz="0" izz="0.1" />
+		</inertial>
+		<collision name="collision">
+			<origin xyz="0 0 0" rpy=" 0 0 0" />
+			<geometry>
+				<box size=".4 .2 .1" />
+			</geometry>
+		</collision>
+		<visual name="chassis_visual">
+			<origin xyz="0 0 0" rpy=" 0 0 0" />
+			<geometry>
+				<box size=".4 .2 .1" />
+			</geometry>
+		</visual>
+		<collision name="back_caster_collision">
+			<origin xyz="-0.15 0 -0.05" rpy=" 0 0 0" />
+			<geometry>
+				<sphere radius="0.0499" />
+			</geometry>
+		</collision>
+		<visual name="back_caster_visual">
+			<origin xyz="-0.15 0 -0.05" rpy=" 0 0 0" />
+			<geometry>
+				<sphere radius="0.05" />
+			</geometry>
+		</visual>
+		<collision name="front_caster_collision">
+			<origin xyz="0.15 0 -0.05" rpy=" 0 0 0" />
+			<geometry>
+				<sphere radius="0.0499" />
+			</geometry>
+		</collision>
+		<visual name="front_caster_visual">
+			<origin xyz="0.15 0 -0.05" rpy=" 0 0 0" />
+			<geometry>
+				<sphere radius="0.05" />
+			</geometry>
+		</visual>
+	</link>
+	<link name="left_wheel">
+		<inertial>
+			<mass value="5.0" />
+			<origin xyz="0 0 0" rpy="0 1.5707 1.5707" />
+			<inertia ixx="0.1" ixy="0" ixz="0" iyy="0.1" iyz="0" izz="0.1" />
+		</inertial>
+		<collision>
+			<origin xyz="0 0 0" rpy="0 1.5707 1.5707" />
+			<geometry>
+				<cylinder radius="0.1" length="0.05" />
+			</geometry>
+		</collision>
+		<visual>
+			<origin xyz="0 0 0" rpy="0 1.5707 1.5707" />
+			<geometry>
+				<cylinder radius="0.1" length="0.05" />
+			</geometry>
+		</visual>
+	</link>
+	<link name="right_wheel">
+		<inertial>
+			<mass value="5.0" />
+			<origin xyz="0 0 0" rpy="0 1.5707 1.5707" />
+			<inertia ixx="0.1" ixy="0" ixz="0" iyy="0.1" iyz="0" izz="0.1" />
+		</inertial>
+		<collision>
+			<origin xyz="0 0 0" rpy="0 1.5707 1.5707" />
+			<geometry>
+				<cylinder radius="0.1" length="0.05" />
+			</geometry>
+		</collision>
+		<visual>
+			<origin xyz="0 0 0" rpy="0 1.5707 1.5707" />
+			<geometry>
+				<cylinder radius="0.1" length="0.05" />
+			</geometry>
+		</visual>
+	</link>
+	<joint type="continuous" name="left_wheel_hinge">
+		<origin xyz="0 0.15 0" rpy="0 0 0" />
+		<child link="left_wheel" />
+		<parent link="chassis" />
+		<axis xyz="0 1 0" rpy="0 0 0" />
+		<limit effort="10000" velocity="1000" />
+		<dynamics damping="1.0" friction="1.0" />
+	</joint>
+	<joint type="continuous" name="right_wheel_hinge">
+		<origin xyz="0 -0.15 0" rpy="0 0 0" />
+		<child link="right_wheel" />
+		<parent link="chassis" />
+		<axis xyz="0 1 0" rpy="0 0 0" />
+		<limit effort="10000" velocity="1000" />
+		<dynamics damping="1.0" friction="1.0" />
+	</joint>
+	<!-- Camera -->
+	<link name="camera">
+		<collision>
+			<origin xyz="0 0 0" rpy="0 0 0" />
+			<geometry>
+				<box size="0.05, 0.05, 0.05" />
+			</geometry>
+		</collision>
+		<visual>
+			<origin xyz="0 0 0" rpy="0 0 0" />
+			<geometry>
+				<box size="0.05, 0.05, 0.05" />
+			</geometry>
+			<material name="red" />
+		</visual>
+		<inertial>
+			<mass value="0.1" />
+			<origin xyz="0 0 0" rpy="0 0 0" />
+			<inertia ixx="1e-6" ixy="0" ixz="0" iyy="1e-6" iyz="0" izz="1e-6" />
+		</inertial>
+	</link>
+	<joint name="camera_joint" type="fixed">
+		<axis xyz="0 1 0" />
+		<origin xyz="0.2 0 0" rpy="0 0 0" />
+		<parent link="chassis" />
+		<child link="camera" />
+	</joint>
+	<link name="hokuyo">
+		<inertial>
+			<mass value="1e-5" />
+			<inertia ixx="1e-6" ixy="0" ixz="0" iyy="1e-6" iyz="0" izz="1e-6" />
+		</inertial>
+		<collision>
+			<origin xyz="0 0 0" rpy="0 0 0" />
+			<geometry>
+				<box size="0.1 0.1 0.1" />
+			</geometry>
+		</collision>
+		<visual>
+			<origin xyz="0 0 0" rpy="0 0 0" />
+			<geometry>
+				<mesh filename="package://my_robot/meshes/hokuyo.dae" />
+			</geometry>
+		</visual>
+	</link>
+	<joint name="hokuyo" type="fixed">
+		<origin xyz="0.15 0 0.1" rpy="0 0 0" />
+		<parent link="chassis" />
+		<child link="hokuyo" />
+    <axis xyz="0 1 0" />
+	</joint>
 </robot>

Commit message: Odom is not displayed

File: src/my_robot/urdf/my_robot.xacro (robot description, xacro)
@@ -2,4 +2,13 @@
 <robot name="my_robot" xmlns:xacro="http://www.ros.org/wiki/xacro">
 	<include filename="$(find my_robot)/urdf/my_robot.gazebo" />
+	<gazebo reference="chassis">
+		<material>Gazebo/FlatBlack</material>
+	</gazebo>
+	<gazebo reference="right_wheel">
+		<material>Gazebo/Orange</material>
+	</gazebo>
+	<gazebo reference="left_wheel">
+		<material>Gazebo/Orange</material>
+	</gazebo>
 	<link name="robot_footprint">
 	</link>
@@ -21,5 +30,5 @@
 			<origin xyz="0 0 0" rpy=" 0 0 0" />
 			<geometry>
-				<box size=".4 .2 .1" />
+				<box size=".4 .24 .13" />
 			</geometry>
 		</collision>
@@ -27,5 +36,5 @@
 			<origin xyz="0 0 0" rpy=" 0 0 0" />
 			<geometry>
-				<box size=".4 .2 .1" />
+				<box size=".4 .24 .13" />
 			</geometry>
 		</visual>
@@ -72,4 +81,7 @@
 				<cylinder radius="0.1" length="0.05" />
 			</geometry>
+			<material name="">
+				<color rgba="0.75294 0.75294 0.75294 1"/>
+			  </material>
 		</visual>
 	</link>
@@ -91,4 +103,7 @@
 				<cylinder radius="0.1" length="0.05" />
 			</geometry>
+			<material name="">
+				<color rgba="0.75294 0.75294 0.75294 1"/>
+			</material>
 		</visual>
 	</link>
@@ -114,5 +129,5 @@
 			<origin xyz="0 0 0" rpy="0 0 0" />
 			<geometry>
-				<box size="0.05, 0.05, 0.05" />
+				<box size="0.05 0.05 0.05" />
 			</geometry>
 		</collision>
@@ -120,5 +135,5 @@
 			<origin xyz="0 0 0" rpy="0 0 0" />
 			<geometry>
-				<box size="0.05, 0.05, 0.05" />
+				<box size="0.05 0.05 0.05" />
 			</geometry>
 			<material name="red" />

Commit message: Can't change color of the camera in RViz

File: src/my_robot/urdf/my_robot.xacro (robot description, xacro)
@@ -1,5 +1,5 @@
 <?xml version="1.0"?>
 <robot name="my_robot" xmlns:xacro="http://www.ros.org/wiki/xacro">
-	<include filename="$(find my_robot)/urdf/my_robot.gazebo" />
+	<xacro:include filename="$(find my_robot)/urdf/my_robot.gazebo" />
 	<gazebo reference="chassis">
 		<material>Gazebo/FlatBlack</material>
@@ -11,6 +11,5 @@
 		<material>Gazebo/Orange</material>
 	</gazebo>
-	<link name="robot_footprint">
-	</link>
+	<link name="robot_footprint"></link>
 	<joint name="robot_footprint_joint" type="fixed">
 		<origin xyz="0 0 0" rpy="0 0 0" />
@@ -82,6 +81,6 @@
 			</geometry>
 			<material name="">
-				<color rgba="0.75294 0.75294 0.75294 1"/>
-			  </material>
+				<color rgba="0.75294 0.75294 0.75294 1" />
+			</material>
 		</visual>
 	</link>
@@ -104,5 +103,5 @@
 			</geometry>
 			<material name="">
-				<color rgba="0.75294 0.75294 0.75294 1"/>
+				<color rgba="0.75294 0.75294 0.75294 1" />
 			</material>
 		</visual>
@@ -173,5 +172,5 @@
 		<parent link="chassis" />
 		<child link="hokuyo" />
-    <axis xyz="0 1 0" />
+		<axis xyz="0 1 0" />
 	</joint>
 </robot>
